Commit message: Add in 6dof joints/links template, modify the first two to look like the physical one

File: kinematics/sixdof_arm.urdf (robot description, URDF)
Before this commit: robot arjan-sixdof-arm, 1 links, 0 joints
Links:
- added link link1; visual box size=1 3 12.2
- added link link2; visual box size=0.1 0.3 0.1
Joints:
- added joint shoulder_lift_joint: type revolute, parent link1, child link2, origin xyz=0 0 0.1 rpy=0 0 0, axis 0 1 0, limit lower=-3.14159 upper=3.14159 effort=100 velocity=3.14
- added joint shoulder_pan_joint: type revolute, parent base_link, child link1, origin xyz=0 0 0 rpy=0 0 0, axis 0 0 1, limit lower=-3.14159 upper=3.14159 effort=100 velocity=3.14

Commit message: Add link2

File: kinematics/sixdof_arm.urdf (robot description, URDF)
Before this commit: robot six_dof_robotic_arm, 3 links, 2 joints
Links:
- link base_link: geometry visual box size=9.0 9.0 2.9
- link link1: geometry visual box size=2.5 2.5 12.2
- link link2: geometry visual box size=6 13 2.5
Joints:
- removed joint shoulder_lift_joint
- removed joint shoulder_pan_joint
- added joint joint1: type revolute, parent base_link, child link1, origin xyz=0 0 0 rpy=0 0 0, axis 0 0 1, limit lower=-1.5707 upper=1.5707 effort=100 velocity=3.14
- added joint joint2: type revolute, parent link1, child link2, origin xyz=0 -1.5 15.1 rpy=0 0 0, axis 1 0 0, limit lower=-1.5707 upper=1.5707 effort=100 velocity=3.14

Commit message: Attempt to move joint 2 axis

File: kinematics/sixdof_arm.urdf (robot description, URDF)
Before this commit: robot six_dof_robotic_arm, 3 links, 2 joints
Links:
- added link link3; visual box size=6 13 2.5
Joints:
- added joint joint3: type revolute, parent link2, child link3, origin xyz=0.4 -13 0 rpy=0 0 0, axis 0 0 1, limit lower=-3.14159 upper=3.14159 effort=100 velocity=3.14
- joint joint1: limit lower=-1.5707 upper=1.5707 effort=100 velocity=3.14 -> lower=-1.57079 upper=1.57079 effort=100 velocity=3.14
- joint joint2: axis 1 0 0 -> -1 0 0; limit lower=-1.5707 upper=1.5707 effort=100 velocity=3.14 -> lower=0 upper=3.14159 effort=100 velocity=3.14; origin xyz=0 -1.5 15.1 rpy=0 0 0 -> xyz=0 11.5 15.1 rpy=0 0 0

Commit message: Get joint 2 placed correctly

File: kinematics/sixdof_arm.urdf (robot description, URDF)
Before this commit: robot six_dof_robotic_arm, 4 links, 3 joints
Links:
- link link1: geometry visual box size=2.5 6.5 12.2
Joints:
- joint joint2: axis -1 0 0 -> 1 0 0; limit lower=0 upper=3.14159 effort=100 velocity=3.14 -> lower=0 upper=3.66519 effort=100 velocity=3.14; origin xyz=0 11.5 15.1 rpy=0 0 0 -> xyz=0 0 14 rpy=0 0 0

Commit message: Model joint3 somewhat closely and re-calibrate robot properties to be more accurate for actuation and angle range

File: kinematics/sixdof_arm.urdf (robot description, URDF)
Before this commit: robot six_dof_robotic_arm, 4 links, 3 joints
Joints:
- joint joint3: axis 0 0 1 -> -1 0 0; limit lower=-3.14159 upper=3.14159 effort=100 velocity=3.14 -> lower=0 upper=3.14159 effort=100 velocity=3.14; origin xyz=0.4 -13 0 rpy=0 0 0 -> xyz=0 13 0 rpy=0.785398 0 0

Commit message: Reduce starting angle roll offset for joint 3

File: kinematics/sixdof_arm.urdf (robot description, URDF)
Before this commit: robot six_dof_robotic_arm, 4 links, 3 joints
Joints:
- joint joint3: origin xyz=0 13 0 rpy=0.785398 0 0 -> xyz=0 13 0 rpy=0.174533 0 0

Commit message: Begin modeling joint4 in URDF

File: kinematics/sixdof_arm.urdf (robot description, URDF)
Before this commit: robot six_dof_robotic_arm, 4 links, 3 joints
Links:
- added link link4; visual box size=3.5 4.25 2.5
Joints:
- added joint joint4: type revolute, parent link3, child link4, origin xyz=0 13 1.25 rpy=1.57079 0 0, axis -1 0 0, limit lower=-3.14159 upper=3.14159 effort=100 velocity=3.14

Commit message: Remove height offset of joint axis in joint4 urdf

File: kinematics/sixdof_arm.urdf (robot description, URDF)
Before this commit: robot six_dof_robotic_arm, 5 links, 4 joints
Joints:
- joint joint4: origin xyz=0 13 1.25 rpy=1.57079 0 0 -> xyz=0 13 0 rpy=1.57079 0 0

Commit message: Make joint4 urdf look like the physical thing

File: kinematics/sixdof_arm.urdf (robot description, URDF)
Before this commit: robot six_dof_robotic_arm, 5 links, 4 joints
Joints:
- joint joint4: origin xyz=0 13 0 rpy=1.57079 0 0 -> xyz=0 11.85 0 rpy=1.57079 0 0

Commit message: Add 5th link and gripper to urdf

File: kinematics/sixdof_arm.urdf (robot description, URDF)
Before this commit: robot six_dof_robotic_arm, 5 links, 4 joints
Links:
- added link gripper_link; visual box size=7.75 11 1.5
- added link link5; visual box size=4.25 3.5 2.5
Joints:
- added joint joint5: type revolute, parent link5, child gripper_link, origin xyz=0 10.5 2.5 rpy=0 0 0, axis 0 1 0, limit lower=-3.14159 upper=3.14159 effort=100 velocity=3.14
- added joint wrist_fixed_joint: type fixed, parent link4, child link5, origin xyz=0.2 0 0 rpy=0 0 0, axis 0 0 1, limit lower=-3.14159 upper=3.14159 effort=100 velocity=3.14

Commit message: Fix joint1 angle limits and have joint5 start at 0

File: kinematics/sixdof_arm.urdf (robot description, URDF)
Before this commit: robot six_dof_robotic_arm, 7 links, 6 joints
Joints:
- joint joint1: limit lower=-1.57079 upper=1.57079 effort=100 velocity=3.14 -> lower=0 upper=3.14159 effort=100 velocity=3.14; origin xyz=0 0 0 rpy=0 0 0 -> xyz=0 0 0 rpy=0 0 -1.570795
- joint joint5: limit lower=-3.14159 upper=3.14159 effort=100 velocity=3.14 -> lower=0 upper=3.14159 effort=100 velocity=3.14

Commit message: Rewrite the ikpy model script to calculate inverse/forward kinematics

File: kinematics/sixdof_arm.urdf (robot description, URDF)
Before this commit: robot six_dof_robotic_arm, 7 links, 6 joints
Joints:
- joint wrist_fixed_joint: axis 0 0 1 -> (none)
